File: motorcontrol/BTN8982_Motor_Control_Shield_Rev_1.0.sch (KiCad schematic (older format))
At the start: 25 parts

Commit message: Add files via upload
Parts:
- BTN8982_DEV.1, BTN8982_DEV.2: footprint BTN8982_Motor_Control_Shield_Rev_1.0:HW-INFINEON_TO263-7-1 -> Package_TO_SOT_SMD:TO-263-6
- C1, C10, C11, C12, C2, C3, C5, C6, C8, C9: footprint BTN8982_Motor_Control_Shield_Rev_1.0:0603-CAP -> Capacitor_SMD:C_0603_1608Metric
- C4: footprint BTN8982_Motor_Control_Shield_Rev_1.0:RCL_E5-13 -> Capacitor_THT:C_Radial_D16.0mm_H25.0mm_P7.50mm
- D2: footprint BTN8982_Motor_Control_Shield_Rev_1.0:SMD-PACKAGES_MELF-D -> Diode_SMD:D_MELF
- R1, R2, R3, R4, R5, R6, R7, R9: footprint BTN8982_Motor_Control_Shield_Rev_1.0:0603-RES -> Resistor_SMD:R_0603_1608Metric
- R10, R8: footprint (none) -> Resistor_SMD:R_0603_1608Metric
- SHAPE1: footprint BTN8982_Motor_Control_Shield_Rev_1.0:XMC1100_FOR_ARDUINO -> (none)
Changed lines of the file:
@@
 F 0 "BTN8982_DEV.1" H 7000 8970 70  0000 L BNN
 F 1 "HW-INFINEON_BTN8982" H 7001 7150 70  0000 L BNN
-F 2 "BTN8982_Motor_Control_Shield_Rev_1.0:HW-INFINEON_TO263-7-1" H 7390 7940 65  0001 L TNN
+F 2 "Package_TO_SOT_SMD:TO-263-6" H 7390 7940 65  0001 L TNN
 F 3 "" H 7400 8150 50  0001 C CNN
 	1    7400 8150
@@
 F 0 "BTN8982_DEV.2" H 14200 8970 70  0000 L BNN
 F 1 "HW-INFINEON_BTN8982" H 14201 7150 70  0000 L BNN
-F 2 "BTN8982_Motor_Control_Shield_Rev_1.0:HW-INFINEON_TO263-7-1" H 14590 7940 65  0001 L TNN
+F 2 "Package_TO_SOT_SMD:TO-263-6" H 14590 7940 65  0001 L TNN
 F 3 "" H 14600 8150 50  0001 C CNN
 	1    14600 8150
@@
 F 0 "C1" H 6360 8965 70  0000 L BNN
 F 1 "100n" H 6360 8765 70  0000 L BNN
-F 2 "BTN8982_Motor_Control_Shield_Rev_1.0:0603-CAP" H 6290 8640 65  0001 L TNN
+F 2 "Capacitor_SMD:C_0603_1608Metric" H 6290 8640 65  0001 L TNN
 F 3 "" H 6300 8850 50  0001 C CNN
 	1    6300 8850
@@
 F 0 "C2" H 13759 8365 70  0000 L BNN
 F 1 "220n" H 13760 8165 70  0000 L BNN
-F 2 "BTN8982_Motor_Control_Shield_Rev_1.0:0603-CAP" H 13690 8040 65  0001 L TNN
+F 2 "Capacitor_SMD:C_0603_1608Metric" H 13690 8040 65  0001 L TNN
 F 3 "" H 13700 8250 50  0001 C CNN
 	1    13700 8250
@@
 F 0 "C3" H 13560 8965 70  0000 L BNN
 F 1 "100n" H 13560 8765 70  0000 L BNN
-F 2 "BTN8982_Motor_Control_Shield_Rev_1.0:0603-CAP" H 13490 8640 65  0001 L TNN
+F 2 "Capacitor_SMD:C_0603_1608Metric" H 13490 8640 65  0001 L TNN
 F 3 "" H 13500 8850 50  0001 C CNN
 	1    13500 8850
@@
 F 0 "C4" H 12145 7668 70  0000 L BNN
 F 1 "1000u" H 12144 7469 70  0000 L BNN
-F 2 "BTN8982_Motor_Control_Shield_Rev_1.0:RCL_E5-13" H 12090 7440 65  0001 L TNN
+F 2 "Capacitor_THT:C_Radial_D16.0mm_H25.0mm_P7.50mm" H 12090 7440 65  0001 L TNN
 F 3 "" H 12100 7650 50  0001 C CNN
 	1    12100 7650
@@
 F 0 "C5" H 6559 8365 70  0000 L BNN
 F 1 "220n" H 6560 8165 70  0000 L BNN
-F 2 "BTN8982_Motor_Control_Shield_Rev_1.0:0603-CAP" H 6490 8040 65  0001 L TNN
+F 2 "Capacitor_SMD:C_0603_1608Metric" H 6490 8040 65  0001 L TNN
 F 3 "" H 6500 8250 50  0001 C CNN
 	1    6500 8250
@@
 F 0 "C6" H 6760 8665 70  0000 L BNN
 F 1 "220n" H 6759 8465 70  0000 L BNN
-F 2 "BTN8982_Motor_Control_Shield_Rev_1.0:0603-CAP" H 6690 8340 65  0001 L TNN
+F 2 "Capacitor_SMD:C_0603_1608Metric" H 6690 8340 65  0001 L TNN
 F 3 "" H 6700 8550 50  0001 C CNN
 	1    6700 8550
@@
 F 0 "C8" H 13960 8665 70  0000 L BNN
 F 1 "220n" H 13959 8465 70  0000 L BNN
-F 2 "BTN8982_Motor_Control_Shield_Rev_1.0:0603-CAP" H 13890 8340 65  0001 L TNN
+F 2 "Capacitor_SMD:C_0603_1608Metric" H 13890 8340 65  0001 L TNN
 F 3 "" H 13900 8550 50  0001 C CNN
 	1    13900 8550
@@
 F 0 "C9" H 15660 7565 70  0000 L BNN
 F 1 "1n" H 15660 7365 70  0000 L BNN
-F 2 "BTN8982_Motor_Control_Shield_Rev_1.0:0603-CAP" H 15590 7240 65  0001 L TNN
+F 2 "Capacitor_SMD:C_0603_1608Metric" H 15590 7240 65  0001 L TNN
 F 3 "" H 15600 7450 50  0001 C CNN
 	1    15600 7450
@@
 F 0 "C10" H 8460 7565 70  0000 L BNN
 F 1 "1n" H 8460 7365 70  0000 L BNN
-F 2 "BTN8982_Motor_Control_Shield_Rev_1.0:0603-CAP" H 8390 7240 65  0001 L TNN
+F 2 "Capacitor_SMD:C_0603_1608Metric" H 8390 7240 65  0001 L TNN
 F 3 "" H 8400 7450 50  0001 C CNN
 	1    8400 7450
@@
 F 0 "C11" H 8359 8265 70  0000 L BNN
 F 1 "100n" H 8360 8066 70  0000 L BNN
-F 2 "BTN8982_Motor_Control_Shield_Rev_1.0:0603-CAP" H 8290 7940 65  0001 L TNN
+F 2 "Capacitor_SMD:C_0603_1608Metric" H 8290 7940 65  0001 L TNN
 F 3 "" H 8300 8150 50  0001 C CNN
 	1    8300 8150
@@
 F 0 "C12" H 15559 8265 70  0000 L BNN
 F 1 "100n" H 15560 8066 70  0000 L BNN
-F 2 "BTN8982_Motor_Control_Shield_Rev_1.0:0603-CAP" H 15490 7940 65  0001 L TNN
+F 2 "Capacitor_SMD:C_0603_1608Metric" H 15490 7940 65  0001 L TNN
 F 3 "" H 15500 8150 50  0001 C CNN
 	1    15500 8150
@@
 F 0 "D2" H 11684 7854 70  0000 L BNN
 F 1 "39V" H 11624 7573 70  0000 L BNN
-F 2 "BTN8982_Motor_Control_Shield_Rev_1.0:SMD-PACKAGES_MELF-D" H 11790 7540 65  0001 L TNN
+F 2 "Diode_SMD:D_MELF" H 11790 7540 65  0001 L TNN
 F 3 "" H 11800 7750 50  0001 C CNN
 	1    11800 7750
@@
 F 0 "R1" H 11650 5709 70  0000 L BNN
 F 1 "10k" H 11650 5520 70  0000 L BNN
-F 2 "BTN8982_Motor_Control_Shield_Rev_1.0:0603-RES" H 11790 5440 65  0001 L TNN
+F 2 "Resistor_SMD:R_0603_1608Metric" H 11790 5440 65  0001 L TNN
 F 3 "" H 11800 5650 50  0001 C CNN
 	1    11800 5650
@@
 F 0 "R2" H 11650 4809 70  0000 L BNN
 F 1 "10k" H 11650 4620 70  0000 L BNN
-F 2 "BTN8982_Motor_Control_Shield_Rev_1.0:0603-RES" H 11790 4540 65  0001 L TNN
+F 2 "Resistor_SMD:R_0603_1608Metric" H 11790 4540 65  0001 L TNN
 F 3 "" H 11800 4750 50  0001 C CNN
 	1    11800 4750
@@
 F 0 "R3" H 12450 4609 70  0000 L BNN
 F 1 "10k" H 12450 4420 70  0000 L BNN
-F 2 "BTN8982_Motor_Control_Shield_Rev_1.0:0603-RES" H 12590 4340 65  0001 L TNN
+F 2 "Resistor_SMD:R_0603_1608Metric" H 12590 4340 65  0001 L TNN
 F 3 "" H 12600 4550 50  0001 C CNN
 	1    12600 4550
@@
 F 0 "R4" H 15350 7708 70  0000 L BNN
 F 1 "1k" H 15350 7520 70  0000 L BNN
-F 2 "BTN8982_Motor_Control_Shield_Rev_1.0:0603-RES" H 15490 7440 65  0001 L TNN
+F 2 "Resistor_SMD:R_0603_1608Metric" H 15490 7440 65  0001 L TNN
 F 3 "" H 15500 7650 50  0001 C CNN
 	1    15500 7650
@@
 F 0 "R5" H 12050 4709 70  0000 L BNN
 F 1 "10k" H 12050 4520 70  0000 L BNN
-F 2 "BTN8982_Motor_Control_Shield_Rev_1.0:0603-RES" H 12190 4440 65  0001 L TNN
+F 2 "Resistor_SMD:R_0603_1608Metric" H 12190 4440 65  0001 L TNN
 F 3 "" H 12200 4650 50  0001 C CNN
 	1    12200 4650
@@
 F 0 "R6" H 15350 8008 70  0000 L BNN
 F 1 "0.51k" H 15350 7820 70  0000 L BNN
-F 2 "BTN8982_Motor_Control_Shield_Rev_1.0:0603-RES" H 15490 7740 65  0001 L TNN
+F 2 "Resistor_SMD:R_0603_1608Metric" H 15490 7740 65  0001 L TNN
 F 3 "" H 15500 7950 50  0001 C CNN
 	1    15500 7950
@@
 F 0 "R7" H 8150 7708 70  0000 L BNN
 F 1 "1k" H 8150 7520 70  0000 L BNN
-F 2 "BTN8982_Motor_Control_Shield_Rev_1.0:0603-RES" H 8290 7440 65  0001 L TNN
+F 2 "Resistor_SMD:R_0603_1608Metric" H 8290 7440 65  0001 L TNN
 F 3 "" H 8300 7650 50  0001 C CNN
 	1    8300 7650
@@
 F 0 "R9" H 8150 8008 70  0000 L BNN
 F 1 "0.51k" H 8150 7820 70  0000 L BNN
-F 2 "BTN8982_Motor_Control_Shield_Rev_1.0:0603-RES" H 8290 7740 65  0001 L TNN
+F 2 "Resistor_SMD:R_0603_1608Metric" H 8290 7740 65  0001 L TNN
 F 3 "" H 8300 7950 50  0001 C CNN
 	1    8300 7950
@@
 F 0 "SHAPE1" V 9200 3900 70  0000 L TNN
 F 1 "ARDUINO_SHIELD" V 9350 3900 70  0000 L TNN
-F 2 "BTN8982_Motor_Control_Shield_Rev_1.0:XMC1100_FOR_ARDUINO" H 9390 3740 65  0001 L TNN
+F 2 "" H 9390 3740 65  0001 L TNN
 F 3 "" H 9400 3950 50  0001 C CNN
 	1    9400 3950
@@
 F 0 "R8" H 10230 8054 50  0000 R CNN
 F 1 "10K" H 10230 8145 50  0000 R CNN
-F 2 "" V 10230 8100 50  0001 C CNN
+F 2 "Resistor_SMD:R_0603_1608Metric" V 10230 8100 50  0001 C CNN
 F 3 "~" H 10300 8100 50  0001 C CNN
 	1    10300 8100
@@
 F 0 "R10" V 10350 8250 50  0000 C CNN
 F 1 "1k" V 10550 8250 50  0000 C CNN
-F 2 "" V 10380 8250 50  0001 C CNN
+F 2 "Resistor_SMD:R_0603_1608Metric" V 10380 8250 50  0001 C CNN
 F 3 "~" H 10450 8250 50  0001 C CNN
 	1    10450 8250
